File: MultiF-Board/MultiF-Board.sch (KiCad schematic (older format))
At the start: 93 parts, among them P1 SERIAL1, P2 SERIAL2, P3 IDE, P4 IDE_LED, U1 74LS14, U10 MMU_GAL, U11 7489, U12 7489, U13 74LS245, U14 74LS90, U15 74LS244, U16 74LS240, U17 TI16550, U18 SRAM_512K, U19 74LS138, U2 8255, U20 MAX-232, U21 SRAM_512K, U22 74LS32, U23 MEM_GAL, U24 74LS06, U25 29EE020, U26 TI16550, U27 74LS244, U28 Z80-CTC, U29 MAX-232, U3 74LS244, U4 74LS244, U5 74LS244, U6 74LS14, U7 74LS32, U8 74LS11, U9 74LS245

Commit message: fdisk 1.1, MultiF-Board schematic upgrade
Parts:
- removed JP3: IDE_VCC, Pin_Headers:Pin_Header_Straight_1x02, symbol JUMPER
- removed JP5: PINHD-2X4, Pin_Headers:Pin_Header_Straight_2x04, symbol PINHD-2X4
- removed unit 1 of U22
- removed unit 3 of U6
- added unit 1 of U22
- added unit 4 of U22
- added unit 4 of U6
- C1, C10, C2, C3, C4, C5, C6, C7, C8, C9: footprint Capacitors_ThroughHole:C_Radial_D5_L6_P2.5 -> Cap2.5; symbol CP-RESCUE-MultiF-Board -> MultiF-Board-rescue:CP-RESCUE-MultiF-Board
- C11, C42: footprint Capacitors_ThroughHole:C_Radial_D6.3_L11.2_P2.5 -> (none); symbol CP1-RESCUE-MultiF-Board -> MultiF-Board-rescue:CP1-RESCUE-MultiF-Board
- C12, C13, C14, C15, C16, C17, C18, C19, C20, C21, C22, C23, C24, C25, C26, C27, C28, C29, C30, C31, C32, C33, C34, C35, C36, C37, C38, C39, C40, C41: footprint Capacitors_ThroughHole:C_Rect_L7_W2.5_P5 -> (none); symbol C-RESCUE-MultiF-Board -> MultiF-Board-rescue:C-RESCUE-MultiF-Board
- D1: symbol LED-RESCUE-MultiF-Board -> MultiF-Board-rescue:LED-RESCUE-MultiF-Board
- JP1, JP2: symbol PINHD-1X3 -> MultiF-Board-rescue:PINHD-1X3
- JPA1, JPB1: symbol PINHD-1X24 -> MultiF-Board-rescue:PINHD-1X24
- P1, P2: symbol CONN_5X2 -> MultiF-Board-rescue:CONN_5X2
- P3: symbol CONN_20X2 -> MultiF-Board-rescue:CONN_20X2
- P4: symbol CONN_2 -> MultiF-Board-rescue:CONN_2
- QG1: symbol OSC -> MultiF-Board-rescue:OSC
- R1, R10, R2, R3, R4, R5, R6, R7, R8, R9: symbol R-RESCUE-MultiF-Board -> MultiF-Board-rescue:R-RESCUE-MultiF-Board
- U1, U6: symbol 74LS14 -> MultiF-Board-rescue:74LS14
- U10: symbol MMU_GAL -> MultiF-Board-rescue:MMU_GAL
- U11, U12: symbol 7489 -> MultiF-Board-rescue:7489
- U13, U9: symbol 74LS245 -> MultiF-Board-rescue:74LS245
- U14: symbol 74LS90 -> MultiF-Board-rescue:74LS90
- U15, U27, U3, U4, U5: symbol 74LS244 -> MultiF-Board-rescue:74LS244
- U16: symbol 74LS240 -> MultiF-Board-rescue:74LS240
- U17, U26: symbol TI16550 -> MultiF-Board-rescue:TI16550
- U18: symbol SRAM_512K -> MultiF-Board-rescue:SRAM_512K
- U19: symbol 74LS138 -> MultiF-Board-rescue:74LS138
- U2: symbol 8255 -> MultiF-Board-rescue:8255
- U20, U29: symbol MAX-232 -> MultiF-Board-rescue:MAX-232
- U21: symbol SRAM_256K -> MultiF-Board-rescue:SRAM_256K
- U22, U7: symbol 74LS32 -> MultiF-Board-rescue:74LS32
- U23: symbol MEM_GAL -> MultiF-Board-rescue:MEM_GAL
- U24: symbol 74LS06 -> MultiF-Board-rescue:74LS06
- U25: symbol 29EE020 -> MultiF-Board-rescue:29EE020
- U28: symbol Z80-CTC -> MultiF-Board-rescue:Z80-CTC
- U8: symbol 74LS11 -> MultiF-Board-rescue:74LS11
Connections:
- wire segments 418 -> 512
