File: VGA_Board/PropVGA.sch (KiCad schematic (older format))
At the start: 80 parts, among them J1 Conn_02x06, J2 Conn_02x06, J3 Conn_02x06, J4 SD_Card, P1 POWER, P2 BOARD_ID, P3 PROPPLUG, P4 VGA, P5 KEYBOARD, P6 SERIAL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

Commit message: Dual IDE support in sysbios
Parts:
- C1, C17, C2, C20, U8: symbol PropIO-V2-rescue:CP -> PropVGA-rescue:CP-PropIO-V2-rescue
- C10, C12, C13, C14, C15, C16, C3, C4, C5, C6, C7, C8, C9: symbol PropIO-V2-rescue:C -> PropVGA-rescue:C-PropIO-V2-rescue
- C11, C18, C19, C21, C22: symbol PropIO-V2-rescue:CP1 -> PropVGA-rescue:CP1-PropIO-V2-rescue
- D1, D2, D3, D4: symbol PropIO-V2-rescue:LED -> PropVGA-rescue:LED-PropIO-V2-rescue
- F1: symbol PropIO-V2-rescue:FUSE -> PropVGA-rescue:FUSE-PropIO-V2-rescue
- JP1: symbol PropIO-V2-rescue:JUMPER3 -> PropVGA-rescue:JUMPER3-PropIO-V2-rescue
- P1: symbol PropIO-V2-rescue:CONN_3 -> PropVGA-rescue:CONN_3-PropIO-V2-rescue
- P2: symbol PropIO-V2-rescue:CONN_6X2 -> PropVGA-rescue:CONN_6X2-PropIO-V2-rescue
- P3: symbol PropIO-V2-rescue:CONN_4 -> PropVGA-rescue:CONN_4-PropIO-V2-rescue
- P4: symbol PropIO-V2-rescue:DE15 -> PropVGA-rescue:DE15-PropIO-V2-rescue
- P5: symbol PropIO-V2-rescue:CONN_6 -> PropVGA-rescue:CONN_6-PropIO-V2-rescue
- P6: symbol PropIO-V2-rescue:CONN_5X2 -> PropVGA-rescue:CONN_5X2-PropIO-V2-rescue
- R1, R10, R11, R12, R13, R14, R15, R16, R17, R18, R19, R2, R20, R21, R22, R23, R3, R4, R5, R6, R7, R8, R9: symbol PropIO-V2-rescue:R -> PropVGA-rescue:R-PropIO-V2-rescue
- RR1: symbol PropIO-V2-rescue:RR9 -> PropVGA-rescue:RR9-PropIO-V2-rescue
- SP1: symbol PropIO-V2-rescue:SPEAKER -> PropVGA-rescue:SPEAKER-PropIO-V2-rescue
- SW1: symbol PropIO-V2-rescue:SW_PUSH -> PropVGA-rescue:SW_PUSH-PropIO-V2-rescue
- U1: symbol PropIO-V2-rescue:74LS06 -> PropVGA-rescue:74LS06-PropIO-V2-rescue
- U10, U12: symbol PropIO-V2-rescue:74LS241 -> PropVGA-rescue:74LS241-PropIO-V2-rescue
- U11: symbol PropIO-V2-rescue:MAX232 -> PropVGA-rescue:MAX232-PropIO-V2-rescue
- U2: symbol PropIO-V2-rescue:74LS682 -> PropVGA-rescue:74LS682-PropIO-V2-rescue
- U3: symbol PropIO-V2-rescue:24C512 -> PropVGA-rescue:24C512-PropIO-V2-rescue
- U4: symbol PropIO-V2-rescue:P8X32A -> PropVGA-rescue:P8X32A-PropIO-V2-rescue
- U5: symbol PropIO-V2-rescue:74LS04 -> PropVGA-rescue:74LS04-PropIO-V2-rescue
- U6: symbol PropIO-V2-rescue:74LS245 -> PropVGA-rescue:74LS245-PropIO-V2-rescue
- U7: symbol PropIO-V2-rescue:LM7805 -> PropVGA-rescue:LM7805-PropIO-V2-rescue
- U9: symbol PropIO-V2-rescue:74LS74 -> PropVGA-rescue:74LS74-PropIO-V2-rescue
- X1: symbol PropIO-V2-rescue:CRYSTAL -> PropVGA-rescue:CRYSTAL-PropIO-V2-rescue
